File: PCB/ESPY.kicad_pcb (KiCad board)
At the start: 4 copper layers, 39.2 x 60.8 mm, 91 parts, among them J1 Conn_01x15_Socket, J2 USB_C_Receptacle_USB2.0_16P, J3 USB_C_Receptacle_USB2.0_16P, J5 Conn_01x15_Socket, J6 Conn_01x20_Pin, J7 Conn_01x08_Pin, J9 Conn_01x16_Pin, SW1 SW_DPST_x2, U2 TLV62569ADRL, U4 TLV62569ADRL, U5 CH334R, Y1 40Mhz(+/-10ppm), Y3 12Mhz

Commit message: files saved
Parts:
- removed C46: 0.1uF, Capacitor_SMD:C_0402_1005Metric
- removed C47: 10uF, Capacitor_SMD:C_0402_1005Metric
- removed C48: 1u, Capacitor_SMD:C_0402_1005Metric
- removed F1: Fuse, Fuse:Fuse_0402_1005Metric
- removed U5: CH334R, Package_SO:QSOP-16_3.9x4.9mm_P0.635mm
- removed Y3: 12Mhz, Crystal:Crystal_SMD_0603-2Pin_6.0x3.5mm
- added C37: 10uF, Capacitor_SMD:C_0402_1005Metric, F.Cu at (144.4, 72.3)
- added C38: 10uF, Capacitor_SMD:C_0402_1005Metric, F.Cu at (144.4, 71.2)
- added U6: SL2.1A, Package_SO:SOIC-16_4.55x10.3mm_P1.27mm, F.Cu at (139.0, 72.2)
- added Y2: 12Mhz, Crystal:Crystal_SMD_3215-2Pin_3.2x1.5mm, F.Cu at (144.6, 68.6)
- J1, J5: footprint Connector_FFC-FPC:Amphenol_F32Q-1A7x1-11015_1x15-1MP_P0.5mm_Horizontal -> Connector_FFC-FPC:Molex_502244-1530_1x15-1MP_P0.5mm_Horizontal
- L2: footprint Inductor_SMD:L_0402_1005Metric -> Inductor_SMD:L_0603_1608Metric
- W25Q512JVFIQ1: footprint Package_SON:WSON-8-1EP_6x5mm_P1.27mm_EP3.4x4.3mm -> Package_SO:SOIC-16W_7.5x10.3mm_P1.27mm
- moved W25Q512JVFIQ1 11.0 mm to (166.2, 79.0), turned to 0 degrees
- moved R35 3.53 mm to (156.3, 66.0), turned to 180 degrees
- moved L2 2.67 mm to (154.8, 72.0)
Routing:
- net /FLASH_CS: track 8.80 -> 28.0 mm
- net /FLASH_WP: track 6.47 -> 21.8 mm, vias 2 -> 3
- net /FLASH_Q: track 4.59 -> 19.7 mm, vias 0 -> 4
- net /DP2+: track 13.3 -> 26.9 mm, vias 0 -> 2
- net /DP2-: track 13.9 -> 25.6 mm, vias 0 -> 2
- net Net-(U5-XO): track 10.8 -> 0.00 mm
- net VBUS: track 61.4 -> 70.6 mm
- net /FLASH_D: track 14.7 -> 23.5 mm
- net GND: track 177.1 -> 168.7 mm, vias 79 -> 63
- net /GPIO23: track 11.6 -> 18.7 mm
- net Net-(U5-VDD33_{LDO}): track 6.86 -> 0.00 mm
- net /VDDO_PSRAM: track 5.26 -> 11.9 mm, vias 0 -> 2
- net Net-(U5-V5): track 6.50 -> 0.00 mm
- net /DP1+: track 13.3 -> 18.9 mm
- net /DP1-: track 14.0 -> 19.4 mm
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Other:
- outline, holes or cut-outs redrawn
